File: PCB/Template.kicad_pcb (KiCad board)
At the start: 2 copper layers, 65 x 56.5 mm, 5 parts, among them P3 Raspberry_Pi_+_Conn

Commit message: PCB design done?
Parts:
- added REF**: TerminalBlock_Philmore_TB133_03x5mm_Straight, Connectors_Terminal_Blocks:TerminalBlock_Philmore_TB133_03x5mm_Straight, F.Cu at (115.8, 122.0)
- added REF**: TerminalBlock_Philmore_TB133_03x5mm_Straight, Connectors_Terminal_Blocks:TerminalBlock_Philmore_TB133_03x5mm_Straight, F.Cu at (132.4, 122.0)
- added REF**: TerminalBlock_Philmore_TB133_03x5mm_Straight, Connectors_Terminal_Blocks:TerminalBlock_Philmore_TB133_03x5mm_Straight, F.Cu at (148.9, 122.0)
- added REF**: TerminalBlock_Philmore_TB132_02x5mm_Straight, Connectors_Terminal_Blocks:TerminalBlock_Philmore_TB132_02x5mm_Straight, F.Cu at (111.4, 83.3)
- added REF**: BARREL_JACK, Connectors:BARREL_JACK, F.Cu at (108.9, 111.2)
Other:
- outline, holes or cut-outs redrawn
- board text added: "+"
- board text added: "-"
- board text added: "DAT"
- board text added: "gnd"
