File: PCB/StrangerThingsWall.kicad_pcb (KiCad board)
At the start: 2 copper layers, 65 x 56.5 mm, 11 parts, among them P3 Raspberry_Pi_+_Conn

Commit message: PCB done and sent off
Other:
- board text added: "13"
- board text added: "18"
- board text added: "19"
- board text added: "e"
